File: KiCad/soverign/soverign.kicad_sch (KiCad schematic)
At the start: 2 parts, among them U1 NUCLEO-G431KB, U2 TCAN332G

Commit message: Kicad Stuff
Parts:
- removed U2: TCAN332G, symbol Interface_CAN_LIN:TCAN332G
- added C1, C2, C3, C4, C5: C, Capacitor_THT:C_Disc_D5.0mm_W2.5mm_P5.00mm, symbol Device:C
- added D1, D2: BAT54S, Package_TO_SOT_SMD:SOT-23, symbol Diode:BAT54S
- added GNDCH0, GNDCH1, GNDOUT1, SIGCH0, SIGCH1, SIGOUT1: TestPoint, Connector_PinHeader_2.54mm:PinHeader_1x01_P2.54mm_Vertical, symbol Connector:TestPoint
- added H1, H2, H3, H4: MountingHole, MountingHole:MountingHole_2.2mm_M2_DIN965_Pad, symbol Mechanical:MountingHole
- added J1, J2: AudioJack3, Connector_Audio:Jack_3.5mm_CUI_SJ1-3523N_Horizontal, symbol Connector_Audio:AudioJack3
- added J3: Barrel_Jack_Switch, Connector_BarrelJack:BarrelJack_Horizontal, symbol Connector:Barrel_Jack_Switch
- added R1, R2, R3, R4, R5: R, Resistor_THT:R_Axial_DIN0207_L6.3mm_D2.5mm_P10.16mm_Horizontal, symbol Device:R
- added R6, R7: 1K, Resistor_THT:R_Axial_DIN0207_L6.3mm_D2.5mm_P10.16mm_Horizontal, symbol Device:R
- added R9: 100R, Resistor_THT:R_Axial_DIN0207_L6.3mm_D2.5mm_P10.16mm_Horizontal, symbol Device:R
- added S1: PEC12R, PEC12R:PEC12R, symbol PEC12R:PEC12R
- added SW1, SW2: SW_Push, Button_Switch_THT:SW_PUSH-12mm, symbol Switch:SW_Push
- added U2: YAAJ_DCDC_StepDown_LM2596, LM2596:LM2596, symbol LM2596:YAAJ_DCDC_StepDown_LM2596
- added U3: XIITIA-STT796, XIITIA-ST7796:XIITIA-ST7796, symbol XIITIA-ST7796:XIITIA-STT796
- added U4: MCP6021, MCP6021:MCP6021, symbol Simulation_SPICE:OPAMP
- U1: footprint NUCLEO-G431KB:MODULE_NUCLEO-G431KB -> NUCLEO_G431KB:MODULE_NUCLEO-G431KB
Connections:
- net +3.3V: now also D1.2 (K), D2.2 (K), R4.2, R5.2, U3.2 (VCC), U4.5 (V+)
- net GND: now also C1.2, C2.2, C3.2, C4.2, C5.2, D1.1 (A), D2.1 (A), GNDCH0.1, GNDCH1.1, GNDOUT1.1, J1.S, J2.S, J3.2, S1.2, S1.C (COMMON), S1.SH1 (SHIELD), S1.SH2 (SHIELD__1), SW1.2, SW2.2, U2.2 (GND), U2.3 (GND), U3.1 (GND), U4.2 (V-)
- net +7.5V: now reaches U1.CN3_1 (VIN)
- net +7.5V: now also U2.4 (Vout)
- net ADC1_IN2: now reaches U1.CN3_11 (PA1(A1))
- net ADC1_IN2: now also D2.3 (COM), R7.2
- net ADC1_IN1: now reaches U1.CN3_12 (PA0(A0))
- net ADC1_IN1: now also D1.3 (COM), R6.2
- net DISPLAY_SDA: now reaches U1.CN3_6 (PA7(A6))
- net DISPLAY_SDA: now also U3.4 (SDA)
- net DISPLAY_SCL: now reaches U1.CN3_8 (PA5/PB7(A4))
- net DISPLAY_SCL: now also U3.3 (SCL)
- net DAC1_OUT1: now reaches U1.CN3_9 (PA4(A3))
- net DAC1_OUT1: now also U4.3 (+)
- net DISPLAY_CS: now reaches U1.CN4_1 (PA9(D1))
- net DISPLAY_CS: now also U3.7 (CS)
- net DISPLAY_BACKLIGHT: now reaches U1.CN4_12 (PA8(D9))
- net DISPLAY_BACKLIGHT: now also U3.8 (BL)
- net BUTTON_1: now reaches U1.CN4_14 (PB5(D11))
- net BUTTON_1: now also C4.1, R4.1, SW1.1
- net BUTTON_2: now reaches U1.CN4_15 (PB4(D12))
- net BUTTON_2: now also C5.1, R5.1, SW2.1
- net DISPLAY_DC: now reaches U1.CN4_2 (PA10(D0))
- net DISPLAY_DC: now also U3.6 (DC)
- net ENCODER_A: now reaches U1.CN4_7 (PB7(D4))
- net ENCODER_A: now also R2.1
- net ENCODER_B: now reaches U1.CN4_9 (PB6(D6))
- net ENCODER_B: now also R1.1
- net FDCAN1_RX renamed DISPLAY_RST
- net DISPLAY_RST: now also U3.5 (RST)
- net FDCAN1_TX renamed ENCODER_SWITCH
- net ENCODER_SWITCH: now also R3.1
- new net: J3.1, U2.1 (Vin)
- new net: C1.1, R1.2, S1.B (CHANNEL_B)
- new net: J1.T, R6.1, SIGCH0.1
- new net: C2.1, R2.2, S1.A (CHANNEL_A)
- new net: J2.T, R7.1, SIGCH1.1
- new net: R9.2, SIGOUT1.1
- new net: R9.1, U4.1, U4.4 (-)
- new net: C3.1, R3.2, S1.1
- no-connect marks 31 -> 20
Other:
- note added: "Buttons"
- note added: "DAC"
- note added: "Display"
- note added: "Microcontroller"
- note added: "Mounting Holes"
- note added: "Oscilloscope Input Channels"
- note added: "Power Supply"
- note added: "Rotary Encoder"
- moved on the sheet: U1
